File: HW/cfd.sch (KiCad schematic (older format))
At the start: 64 parts

Commit message: update
Other:
- note added: "opt 0R"
- note added: "opt 27R"
- note added: "opt 46R4"
- note removed: "opt 27R4"
Changed lines of the file:
@@
 Sheet 1 1
 Title "Constant Fraction Discriminator"
-Date "26 jun 2013"
+Date "27 jun 2013"
 Rev "0.1"
 Comp "DH consulting"
@@
 opt 8R25
 Text Notes 6000 7500 3    60   ~ 0
-opt 27R4
+opt 27R
 $Comp
 L DGND #PWR?
@@
 	1    0    0    -1
 $EndComp
+Text Notes 6000 8450 3    60   ~ 0
+opt 46R4
+Text Notes 5350 8450 0    60   ~ 0
+opt 0R
 $EndSCHEMATC
